File: hardware/baseboard_4slots/baseboard_4slots.kicad_pcb (KiCad board)
At the start: 2 copper layers, 354 x 60 mm, 37 parts, among them J1 IO-Board_00, J2 IO-Board_01, J3 IO-Board_10, J4 IO-Board_11, J5 USB_B_Micro, J6 Conn_01x05: Adafruit 1833, J7 Screw_Terminal_01x04, J8 Conn_02x02_Odd_Even, J9 Conn_02x02_Odd_Even, U1 NRF24L01_Breakout, U2 Pico

Commit message: Minimal trace routing improvements
Routing:
- net +3V3: track 529.4 -> 530.4 mm
- net GND: vias 238 -> 244
Other:
- net class Default removed
